File: ws2812_2020_8x.sch (KiCad schematic (older format))
At the start: 9 parts

Commit message: Minor updates
Parts:
- D1, D2, D3, D4, D5, D6, D7, D8: symbol LED:WS2812_2020 -> WM_lib:WS2812_2020-LED
Changed lines of the file:
@@
 EESchema Schematic File Version 4
-EELAYER 29 0
+EELAYER 30 0
 EELAYER END
 $Descr A4 11693 8268
 encoding utf-8
-Sheet 2 9
+Sheet 1 1
 Title ""
 Date ""
@@
 $EndDescr
 $Comp
-L LED:WS2812_2020 D1
+L WM_lib:WS2812_2020-LED D1
 U 1 1 5EADECB6
 P 3750 2200
@@
 AR Path="/5EAE355D/5EADECB6" Ref="D49"  Part="1"
 AR Path="/5EAE3563/5EADECB6" Ref="D57"  Part="1"
+AR Path="/5EADECB6" Ref="D1"  Part="1"
 F 0 "D1" H 4094 2246 50  0000 L CNN
 F 1 "WS2812_2020" H 4094 2155 50  0000 L CNN
@@
 $EndComp
 $Comp
-L LED:WS2812_2020 D2
+L WM_lib:WS2812_2020-LED D2
 U 1 1 5EAE1759
 P 4500 2200
@@
 AR Path="/5EAE355D/5EAE1759" Ref="D50"  Part="1"
 AR Path="/5EAE3563/5EAE1759" Ref="D58"  Part="1"
+AR Path="/5EAE1759" Ref="D2"  Part="1"
 F 0 "D2" H 4844 2246 50  0000 L CNN
 F 1 "WS2812_2020" H 4844 2155 50  0000 L CNN
@@
 $EndComp
 $Comp
-L LED:WS2812_2020 D3
+L WM_lib:WS2812_2020-LED D3
 U 1 1 5EAE2ADE
 P 5250 2200
@@
 AR Path="/5EAE355D/5EAE2ADE" Ref="D51"  Part="1"
 AR Path="/5EAE3563/5EAE2ADE" Ref="D59"  Part="1"
+AR Path="/5EAE2ADE" Ref="D3"  Part="1"
 F 0 "D3" H 5594 2246 50  0000 L CNN
 F 1 "WS2812_2020" H 5594 2155 50  0000 L CNN
@@
 $EndComp
 $Comp
-L LED:WS2812_2020 D4
+L WM_lib:WS2812_2020-LED D4
 U 1 1 5EAE2AE4
 P 6000 2200
@@
 AR Path="/5EAE355D/5EAE2AE4" Ref="D52"  Part="1"
 AR Path="/5EAE3563/5EAE2AE4" Ref="D60"  Part="1"
+AR Path="/5EAE2AE4" Ref="D4"  Part="1"
 F 0 "D4" H 6344 2246 50  0000 L CNN
 F 1 "WS2812_2020" H 6344 2155 50  0000 L CNN
@@
 $EndComp
 $Comp
-L LED:WS2812_2020 D5
+L WM_lib:WS2812_2020-LED D5
 U 1 1 5EAE9322
 P 3750 3350
@@
 AR Path="/5EAE355D/5EAE9322" Ref="D53"  Part="1"
 AR Path="/5EAE3563/5EAE9322" Ref="D61"  Part="1"
+AR Path="/5EAE9322" Ref="D5"  Part="1"
 F 0 "D5" H 4094 3396 50  0000 L CNN
 F 1 "WS2812_2020" H 4094 3305 50  0000 L CNN
@@
 $EndComp
 $Comp
-L LED:WS2812_2020 D6
+L WM_lib:WS2812_2020-LED D6
 U 1 1 5EAE9328
 P 4500 3350
@@
 AR Path="/5EAE355D/5EAE9328" Ref="D54"  Part="1"
 AR Path="/5EAE3563/5EAE9328" Ref="D62"  Part="1"
+AR Path="/5EAE9328" Ref="D6"  Part="1"
 F 0 "D6" H 4844 3396 50  0000 L CNN
 F 1 "WS2812_2020" H 4844 3305 50  0000 L CNN
@@
 $EndComp
 $Comp
-L LED:WS2812_2020 D7
+L WM_lib:WS2812_2020-LED D7
 U 1 1 5EAE932E
 P 5250 3350
@@
 AR Path="/5EAE355D/5EAE932E" Ref="D55"  Part="1"
 AR Path="/5EAE3563/5EAE932E" Ref="D63"  Part="1"
+AR Path="/5EAE932E" Ref="D7"  Part="1"
 F 0 "D7" H 5594 3396 50  0000 L CNN
 F 1 "WS2812_2020" H 5594 3305 50  0000 L CNN
@@
 $EndComp
 $Comp
-L LED:WS2812_2020 D8
+L WM_lib:WS2812_2020-LED D8
 U 1 1 5EAE9334
 P 6000 3350
@@
 AR Path="/5EAE355D/5EAE9334" Ref="D56"  Part="1"
 AR Path="/5EAE3563/5EAE9334" Ref="D64"  Part="1"
+AR Path="/5EAE9334" Ref="D8"  Part="1"
 F 0 "D8" H 6344 3396 50  0000 L CNN
 F 1 "WS2812_2020" H 6344 3305 50  0000 L CNN
